Commit message: refactor: update robot model configuration, migrate sensor data scripts, and reorganize launch assets

File: romi_ws/src/romi_gazebo/models/romi_meshes.urdf (robot description, URDF)
Before this commit: robot romi, 8 links, 7 joints
Links:
- link base_link: geometry collision box size=0.16 0.14 0.04; visual mesh filename=package://romi_gazebo/meshes/visual/chasis.stl scale=0.001 0.001 0.001
- link imu_link: geometry collision mesh filename=package://romi_gazebo/meshes/visual/control_board.stl scale=0.001 0.001 0.001; visual mesh filename=package://romi_gazebo/meshes/visual/control_board.stl scale=0.001 0.001 0.001
- link left_wheel: geometry collision cylinder length=0.015 radius=0.035; visual mesh filename=package://romi_gazebo/meshes/visual/wheel.stl scale=0.001 0.001 0.001
- link right_wheel: geometry collision cylinder length=0.015 radius=0.035; visual mesh filename=package://romi_gazebo/meshes/visual/wheel.stl scale=0.001 0.001 0.001
